File: schematics/test2/test2.kicad_sch (KiCad schematic)
At the start: 10 parts, among them SW1 SW_DIP_x08, SW2 SW_DIP_x08, U1 74AUC2G04

Commit message: a lot of stuff
Parts:
- added D10, D11, D12, D13, D14, D15, D16, D17, D2, D3, D4, D5, D6, D7, D8, D9: US1M, Diode_SMD:D_SMA, symbol Diode:US1M
- added MIK1: (no value), symbol cunstom:MIK32_ADC
- added MIK32 (x2): (no value), symbol cunstom:MIK32
- added R1, R10, R11, R12, R2, R3, R4, R5, R6, R7, R8, R9: 10 кОм, symbol Device:R_Small
- added R13, R14: 20k, symbol Device:R
- added RV1, RV2: 10k, symbol Device:R_Potentiometer
- added SW10, SW11, SW12, SW13, SW14, SW15, SW16, SW17, SW18, SW19, SW20, SW5, SW6, SW7, SW8, SW9: SW_Push, symbol Switch:SW_Push
- added SW3: SW_DIP_x08, symbol Switch:SW_DIP_x08
Connections:
- net +3V3: now also MIK1. (GND), MIK32. (GND), MIK32. (GND), R10.1, R11.1, R12.1, R13.1, R14.1, R9.1, SW3.1, SW3.2, SW3.3, SW3.4, SW3.5, SW3.6, SW3.7, SW3.8
- net GND: now also MIK1. (GND), MIK32. (GND), MIK32. (GND), R1.2, R2.2, R3.2, R4.2, R5.2, R6.2, R7.2, R8.2, RV1.1, RV2.1
- new net: MIK32. (GND), R2.1, SW3.10
- new net: MIK32. (GND), R3.1, SW3.11
- new net: MIK32. (GND), R4.1, SW3.12
- new net: MIK32. (GND), R5.1, SW3.13
- new net: MIK32. (GND), R6.1, SW3.14
- new net: MIK32. (GND), R7.1, SW3.15
- new net: MIK32. (GND), R8.1, SW3.16
- new net: MIK32. (GND), R1.1, SW3.9
- new net: MIK32. (GND), R11.2, SW13.1, SW14.1, SW15.1, SW16.1
- new net: D10.2 (A), SW13.2
- new net: MIK32. (GND), R12.2, SW17.1, SW18.1, SW19.1, SW20.1
- new net: D11.2 (A), SW17.2
- new net: D10.1 (K), D11.1 (K), D2.1 (K), D6.1 (K), MIK32. (GND)
- new net: MIK32. (GND), R10.2, SW10.1, SW11.1, SW12.1, SW9.1
- new net: D7.2 (A), SW10.2
- new net: D14.1 (K), D15.1 (K), D4.1 (K), D8.1 (K), MIK32. (GND)
- new net: D8.2 (A), SW11.2
- new net: D16.1 (K), D17.1 (K), D5.1 (K), D9.1 (K), MIK32. (GND)
- new net: D17.2 (A), SW20.2
- new net: MIK1. (GND), RV1.2
- new net: R13.2, RV1.3
- new net: MIK32. (GND), R9.2, SW5.1, SW6.1, SW7.1, SW8.1
- new net: D12.1 (K), D13.1 (K), D3.1 (K), D7.1 (K), MIK32. (GND)
- new net: D12.2 (A), SW14.2
- new net: D3.2 (A), SW6.2
- new net: D2.2 (A), SW5.2
- new net: D13.2 (A), SW18.2
- new net: MIK1. (GND), RV2.2
- new net: D6.2 (A), SW9.2
- new net: D16.2 (A), SW16.2
- new net: D15.2 (A), SW19.2
- new net: D14.2 (A), SW15.2
- new net: D9.2 (A), SW12.2
- new net: D4.2 (A), SW7.2
- new net: R14.2, RV2.3
- new net: D5.2 (A), SW8.2
Other:
- moved on the sheet: 100nF, C1, D1, R1, R2, R3, SW1, SW2
